File: PCB/QS-HUB-DB.kicad_pcb (KiCad board)
At the start: 2 copper layers, 104 x 29.2 mm, 54 parts, among them J1 JST, J3 USB_A, J4 USB_A, J5 USB_C_Receptacle_USB2.0, U1 MIC2026-2BM, U2 FE1.1, U3 USBLC6-2SC6, U4 USBLC6-2SC6, U6 USBLC6-2SC6, Y1 12MHz

Commit message: Added 3D model and updated silk
Other:
- board text added: "https://github.com/Armastardo/QS-HUB-DB"
Changed lines of the file:
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@@
       (rotate (xyz 0 0 0))
     )
+    (model "C:/Users/bbr_b/Documents/MechanicalKeyboards/SM04B-SRSS-TB.STEP"
+      (offset (xyz 0 1.5 0))
+      (scale (xyz 1 1 1))
+      (rotate (xyz -90 0 0))
+    )
   )
   (footprint "Package_TO_SOT_SMD:SOT-23-6" (layer "F.Cu")
@@
   (gr_line (start 177.18 45.894771) (end 79.2 45.894771)
     (stroke (width 0.1) (type default)) (layer "Edge.Cuts"))
+  (gr_text "https://github.com/Armastardo/QS-HUB-DB" (at 175.06 44.01) (layer "B.SilkS")
+    (effects (font (size 1.5 1.5) (thickness 0.3) bold) (justify left bottom mirror))
+  )
   (gr_text "19.99" (at 78.21 33.58 270) (layer "B.SilkS")
     (effects (font (size 1 1) (thickness 0.2) bold) (justify left bottom mirror))
